File: _autosave-usb-ttl.sch (KiCad schematic (older format))
At the start: 9 parts, among them J1 USB_A, J2 Conn_01x05, U1 CH330N

Commit message: update
Parts:
- J1: footprint Heatsink:Heatsink_AAVID_573300D00010G_TO-263 -> HANK:USB_A_HANK
Other:
- moved on the sheet: D1, D2, R1, R2
Changed lines of the file:
@@
 F 0 "J1" H 4457 4167 50  0000 C CNN
 F 1 "USB_A" H 4457 4076 50  0000 C CNN
-F 2 "Heatsink:Heatsink_AAVID_573300D00010G_TO-263" H 4550 3650 50  0001 C CNN
+F 2 "HANK:USB_A_HANK" H 4550 3650 50  0001 C CNN
 F 3 " ~" H 4550 3650 50  0001 C CNN
 	1    4400 3700
@@
 L Device:LED D1
 U 1 1 5EFCB754
-P 8300 4000
-F 0 "D1" V 8400 3950 50  0000 R CNN
-F 1 "LED" V 8248 3882 50  0000 R CNN
-F 2 "LED_SMD:LED_0603_1608Metric" H 8300 4000 50  0001 C CNN
-F 3 "~" H 8300 4000 50  0001 C CNN
-	1    8300 4000
+P 7950 3950
+F 0 "D1" V 8050 3900 50  0000 R CNN
+F 1 "LED" V 7898 3832 50  0000 R CNN
+F 2 "LED_SMD:LED_0603_1608Metric" H 7950 3950 50  0001 C CNN
+F 3 "~" H 7950 3950 50  0001 C CNN
+	1    7950 3950
 	0    -1   1    0
 $EndComp
@@
 RXD
 Wire Wire Line
-	8300 3850 8300 3550
+	7950 3800 7950 3500
 $Comp
 L power:+5V #PWR03
 U 1 1 5EFDCF93
-P 8300 3100
-F 0 "#PWR03" H 8300 2950 50  0001 C CNN
-F 1 "+5V" H 8315 3273 50  0000 C CNN
-F 2 "" H 8300 3100 50  0001 C CNN
-F 3 "" H 8300 3100 50  0001 C CNN
-	1    8300 3100
-	1    0    0    -1
-$EndComp
-Wire Wire Line
-	8300 3100 8300 3250
+P 7950 3050
+F 0 "#PWR03" H 7950 2900 50  0001 C CNN
+F 1 "+5V" H 7965 3223 50  0000 C CNN
+F 2 "" H 7950 3050 50  0001 C CNN
+F 3 "" H 7950 3050 50  0001 C CNN
+	1    7950 3050
+	1    0    0    -1
+$EndComp
+Wire Wire Line
+	7950 3050 7950 3200
 $Comp
 L Device:R R1
 U 1 1 5EFCB28C
-P 8300 3400
-F 0 "R1" H 8370 3446 50  0000 L CNN
-F 1 "4.7k" V 8300 3300 50  0000 L CNN
-F 2 "Resistor_SMD:R_0603_1608Metric" V 8230 3400 50  0001 C CNN
-F 3 "~" H 8300 3400 50  0001 C CNN
-	1    8300 3400
-	1    0    0    -1
-$EndComp
-Text Label 8300 4250 2    50   ~ 0
+P 7950 3350
+F 0 "R1" H 8020 3396 50  0000 L CNN
+F 1 "4.7k" V 7950 3250 50  0000 L CNN
+F 2 "Resistor_SMD:R_0603_1608Metric" V 7880 3350 50  0001 C CNN
+F 3 "~" H 7950 3350 50  0001 C CNN
+	1    7950 3350
+	1    0    0    -1
+$EndComp
+Text Label 7950 4200 2    50   ~ 0
 TXD
 $Comp
 L Device:LED D2
 U 1 1 5EFDED84
-P 8950 4000
-F 0 "D2" V 9050 3950 50  0000 R CNN
-F 1 "LED" V 8898 3882 50  0000 R CNN
-F 2 "LED_SMD:LED_0603_1608Metric" H 8950 4000 50  0001 C CNN
-F 3 "~" H 8950 4000 50  0001 C CNN
-	1    8950 4000
+P 8600 3950
+F 0 "D2" V 8700 3900 50  0000 R CNN
+F 1 "LED" V 8548 3832 50  0000 R CNN
+F 2 "LED_SMD:LED_0603_1608Metric" H 8600 3950 50  0001 C CNN
+F 3 "~" H 8600 3950 50  0001 C CNN
+	1    8600 3950
 	0    -1   -1   0
 $EndComp
 Wire Wire Line
-	8950 3850 8950 3550
+	8600 3800 8600 3500
 $Comp
 L power:+5V #PWR04
 U 1 1 5EFDED8F
-P 8950 3100
-F 0 "#PWR04" H 8950 2950 50  0001 C CNN
-F 1 "+5V" H 8965 3273 50  0000 C CNN
-F 2 "" H 8950 3100 50  0001 C CNN
-F 3 "" H 8950 3100 50  0001 C CNN
-	1    8950 3100
-	1    0    0    -1
-$EndComp
-Wire Wire Line
-	8950 3100 8950 3250
+P 8600 3050
+F 0 "#PWR04" H 8600 2900 50  0001 C CNN
+F 1 "+5V" H 8615 3223 50  0000 C CNN
+F 2 "" H 8600 3050 50  0001 C CNN
+F 3 "" H 8600 3050 50  0001 C CNN
+	1    8600 3050
+	1    0    0    -1
+$EndComp
+Wire Wire Line
+	8600 3050 8600 3200
 $Comp
 L Device:R R2
 U 1 1 5EFDED9A
-P 8950 3400
-F 0 "R2" H 9020 3446 50  0000 L CNN
-F 1 "4.7k" V 8950 3300 50  0000 L CNN
-F 2 "Resistor_SMD:R_0603_1608Metric" V 8880 3400 50  0001 C CNN
-F 3 "~" H 8950 3400 50  0001 C CNN
-	1    8950 3400
+P 8600 3350
+F 0 "R2" H 8670 3396 50  0000 L CNN
+F 1 "4.7k" V 8600 3250 50  0000 L CNN
+F 2 "Resistor_SMD:R_0603_1608Metric" V 8530 3350 50  0001 C CNN
+F 3 "~" H 8600 3350 50  0001 C CNN
+	1    8600 3350
 	1    0    0    1
 $EndComp
-Text Label 8950 4250 2    50   ~ 0
+Text Label 8600 4200 2    50   ~ 0
 RXD
 Wire Wire Line
-	8300 4150 8300 4250
-Wire Wire Line
-	8950 4150 8950 4250
+	7950 4100 7950 4200
+Wire Wire Line
+	8600 4100 8600 4200
 Wire Wire Line
 	4300 4100 4300 4350

Commit message: update
Parts:
- J1: footprint HANK:USB_A_HANK -> HANK:USB_A_CNCTech_1001-011-01101_Horizontal
Other:
- moved on the sheet: D1, D2, R1, R2
Changed lines of the file:
@@
 F 0 "J1" H 4457 4167 50  0000 C CNN
 F 1 "USB_A" H 4457 4076 50  0000 C CNN
-F 2 "HANK:USB_A_HANK" H 4550 3650 50  0001 C CNN
+F 2 "HANK:USB_A_CNCTech_1001-011-01101_Horizontal" H 4550 3650 50  0001 C CNN
 F 3 " ~" H 4550 3650 50  0001 C CNN
 	1    4400 3700
@@
 L Device:LED D1
 U 1 1 5EFCB754
-P 7950 3950
-F 0 "D1" V 8050 3900 50  0000 R CNN
-F 1 "LED" V 7898 3832 50  0000 R CNN
-F 2 "LED_SMD:LED_0603_1608Metric" H 7950 3950 50  0001 C CNN
-F 3 "~" H 7950 3950 50  0001 C CNN
-	1    7950 3950
+P 8300 4000
+F 0 "D1" V 8400 3950 50  0000 R CNN
+F 1 "LED" V 8248 3882 50  0000 R CNN
+F 2 "LED_SMD:LED_0603_1608Metric" H 8300 4000 50  0001 C CNN
+F 3 "~" H 8300 4000 50  0001 C CNN
+	1    8300 4000
 	0    -1   1    0
 $EndComp
@@
 RXD
 Wire Wire Line
-	7950 3800 7950 3500
+	8300 3850 8300 3550
 $Comp
 L power:+5V #PWR03
 U 1 1 5EFDCF93
-P 7950 3050
-F 0 "#PWR03" H 7950 2900 50  0001 C CNN
-F 1 "+5V" H 7965 3223 50  0000 C CNN
-F 2 "" H 7950 3050 50  0001 C CNN
-F 3 "" H 7950 3050 50  0001 C CNN
-	1    7950 3050
-	1    0    0    -1
-$EndComp
-Wire Wire Line
-	7950 3050 7950 3200
+P 8300 3100
+F 0 "#PWR03" H 8300 2950 50  0001 C CNN
+F 1 "+5V" H 8315 3273 50  0000 C CNN
+F 2 "" H 8300 3100 50  0001 C CNN
+F 3 "" H 8300 3100 50  0001 C CNN
+	1    8300 3100
+	1    0    0    -1
+$EndComp
+Wire Wire Line
+	8300 3100 8300 3250
 $Comp
 L Device:R R1
 U 1 1 5EFCB28C
-P 7950 3350
-F 0 "R1" H 8020 3396 50  0000 L CNN
-F 1 "4.7k" V 7950 3250 50  0000 L CNN
-F 2 "Resistor_SMD:R_0603_1608Metric" V 7880 3350 50  0001 C CNN
-F 3 "~" H 7950 3350 50  0001 C CNN
-	1    7950 3350
-	1    0    0    -1
-$EndComp
-Text Label 7950 4200 2    50   ~ 0
+P 8300 3400
+F 0 "R1" H 8370 3446 50  0000 L CNN
+F 1 "4.7k" V 8300 3300 50  0000 L CNN
+F 2 "Resistor_SMD:R_0603_1608Metric" V 8230 3400 50  0001 C CNN
+F 3 "~" H 8300 3400 50  0001 C CNN
+	1    8300 3400
+	1    0    0    -1
+$EndComp
+Text Label 8300 4250 2    50   ~ 0
 TXD
 $Comp
 L Device:LED D2
 U 1 1 5EFDED84
-P 8600 3950
-F 0 "D2" V 8700 3900 50  0000 R CNN
-F 1 "LED" V 8548 3832 50  0000 R CNN
-F 2 "LED_SMD:LED_0603_1608Metric" H 8600 3950 50  0001 C CNN
-F 3 "~" H 8600 3950 50  0001 C CNN
-	1    8600 3950
+P 8950 4000
+F 0 "D2" V 9050 3950 50  0000 R CNN
+F 1 "LED" V 8898 3882 50  0000 R CNN
+F 2 "LED_SMD:LED_0603_1608Metric" H 8950 4000 50  0001 C CNN
+F 3 "~" H 8950 4000 50  0001 C CNN
+	1    8950 4000
 	0    -1   -1   0
 $EndComp
 Wire Wire Line
-	8600 3800 8600 3500
+	8950 3850 8950 3550
 $Comp
 L power:+5V #PWR04
 U 1 1 5EFDED8F
-P 8600 3050
-F 0 "#PWR04" H 8600 2900 50  0001 C CNN
-F 1 "+5V" H 8615 3223 50  0000 C CNN
-F 2 "" H 8600 3050 50  0001 C CNN
-F 3 "" H 8600 3050 50  0001 C CNN
-	1    8600 3050
-	1    0    0    -1
-$EndComp
-Wire Wire Line
-	8600 3050 8600 3200
+P 8950 3100
+F 0 "#PWR04" H 8950 2950 50  0001 C CNN
+F 1 "+5V" H 8965 3273 50  0000 C CNN
+F 2 "" H 8950 3100 50  0001 C CNN
+F 3 "" H 8950 3100 50  0001 C CNN
+	1    8950 3100
+	1    0    0    -1
+$EndComp
+Wire Wire Line
+	8950 3100 8950 3250
 $Comp
 L Device:R R2
 U 1 1 5EFDED9A
-P 8600 3350
-F 0 "R2" H 8670 3396 50  0000 L CNN
-F 1 "4.7k" V 8600 3250 50  0000 L CNN
-F 2 "Resistor_SMD:R_0603_1608Metric" V 8530 3350 50  0001 C CNN
-F 3 "~" H 8600 3350 50  0001 C CNN
-	1    8600 3350
+P 8950 3400
+F 0 "R2" H 9020 3446 50  0000 L CNN
+F 1 "4.7k" V 8950 3300 50  0000 L CNN
+F 2 "Resistor_SMD:R_0603_1608Metric" V 8880 3400 50  0001 C CNN
+F 3 "~" H 8950 3400 50  0001 C CNN
+	1    8950 3400
 	1    0    0    1
 $EndComp
-Text Label 8600 4200 2    50   ~ 0
+Text Label 8950 4250 2    50   ~ 0
 RXD
 Wire Wire Line
-	7950 4100 7950 4200
-Wire Wire Line
-	8600 4100 8600 4200
+	8300 4150 8300 4250
+Wire Wire Line
+	8950 4150 8950 4250
 Wire Wire Line
 	4300 4100 4300 4350
