File: usb-ttl.kicad_pcb (KiCad board)
At the start: 2 copper layers, 25 x 16 mm, 9 parts, among them J1 USB_A, J2 Conn_01x05, U1 CH330N

Commit message: update
Parts:
- J1: footprint Connector_USB:USB_A_CNCTech_1001-011-01101_Horizontal -> HANK:USB_A_HANK

Commit message: update
Parts:
- turned U1 to 90 degrees
Routing:
- added copper zone on B.Cu, net GND
- added copper zone on F.Cu, net GND
Other:
- board text added: "5V"
- board text added: "GND"
- board text added: "RTS"
- board text added: "RXD"
- board text added: "TXD"
- board text added: "https://uinika.gitee.io/"

Commit message: update
Parts:
- J1: footprint HANK:USB_A_HANK -> HANK:USB_A_CNCTech_1001-011-01101_Horizontal
