File: usb-ttl.sch (KiCad schematic (older format))
At the start: 9 parts, among them J1 USB_A, J2 Conn_01x05, U1 CH330N

Commit message: update
Parts:
- J1: footprint Connector_USB:USB_A_CNCTech_1001-011-01101_Horizontal -> HANK:USB_A_HANK
Changed lines of the file:
@@
 F 0 "J1" H 4457 4167 50  0000 C CNN
 F 1 "USB_A" H 4457 4076 50  0000 C CNN
-F 2 "Connector_USB:USB_A_CNCTech_1001-011-01101_Horizontal" H 4550 3650 50  0001 C CNN
+F 2 "HANK:USB_A_HANK" H 4550 3650 50  0001 C CNN
 F 3 " ~" H 4550 3650 50  0001 C CNN
 	1    4400 3700

Commit message: update
Parts:
- J1: footprint HANK:USB_A_HANK -> HANK:USB_A_CNCTech_1001-011-01101_Horizontal
Changed lines of the file:
@@
 F 0 "J1" H 4457 4167 50  0000 C CNN
 F 1 "USB_A" H 4457 4076 50  0000 C CNN
-F 2 "HANK:USB_A_HANK" H 4550 3650 50  0001 C CNN
+F 2 "HANK:USB_A_CNCTech_1001-011-01101_Horizontal" H 4550 3650 50  0001 C CNN
 F 3 " ~" H 4550 3650 50  0001 C CNN
 	1    4400 3700
